File: hardware-KiCad/zynthian-mini.kicad_sch (KiCad schematic)
At the start: 37 parts, among them SW1 SW_Push, SW2 SW_Push, SW3 SW_Push, SW4 SW_Push, U1 74HCT14, U2 H11L1M

Commit message: first button layout try
Parts:
- added C10, C11, C12, C14, C15, C17, C18, C20, C21, C23, C24, C25, C26, C27, C8, C9: 100n, Capacitor_THT:C_Rect_L4.0mm_W2.5mm_P2.50mm, symbol Device:C
- added C7: 100n, Capacitor_THT:C_Rect_L7.0mm_W2.0mm_P5.00mm, symbol Device:C
- added MCPMCP23017_SP2: MCP23017_SP, Package_DIP:DIP-28_W7.62mm, symbol Interface_Expansion:MCP23017_SP
- added R7, R8: 10k, Resistor_THT:R_Axial_DIN0207_L6.3mm_D2.5mm_P7.62mm_Horizontal, symbol Device:R
- added SW10, SW11, SW12, SW13, SW14, SW15, SW16, SW17, SW18, SW19, SW20, SW5, SW6, SW7, SW8, SW9: SW_Push, project-footprints:push-button, symbol Switch:SW_Push
Connections:
- net +3.3V: now also R7.2, R8.2
- net +5V: now also C7.1, MCPMCP23017_SP2.18 (~{RESET}), MCPMCP23017_SP2.9 (VDD)
- net ENC-A-1: now also MCPMCP23017_SP1.1 (GPB0); no longer MCPMCP23017_SP1.22 (GPA1)
- net ENC-A-2: now also MCPMCP23017_SP1.3 (GPB2); no longer MCPMCP23017_SP1.25 (GPA4)
- net ENC-A-3: now also MCPMCP23017_SP1.5 (GPB4); no longer MCPMCP23017_SP1.2 (GPB1)
- net ENC-A-4: now also MCPMCP23017_SP1.7 (GPB6); no longer MCPMCP23017_SP1.5 (GPB4)
- net ENC-B-1: now also MCPMCP23017_SP1.2 (GPB1); no longer MCPMCP23017_SP1.23 (GPA2)
- net ENC-B-2: now also MCPMCP23017_SP1.4 (GPB3); no longer MCPMCP23017_SP1.26 (GPA5)
- net ENC-B-3: now also MCPMCP23017_SP1.6 (GPB5); no longer MCPMCP23017_SP1.3 (GPB2)
- net ENC-B-4: now also MCPMCP23017_SP1.8 (GPB7); no longer MCPMCP23017_SP1.6 (GPB5)
- net ENC-SW-1: now also MCPMCP23017_SP1.25 (GPA4); no longer MCPMCP23017_SP1.21 (GPA0)
- net ENC-SW-2: now also MCPMCP23017_SP1.26 (GPA5); no longer MCPMCP23017_SP1.24 (GPA3)
- net ENC-SW-3: now also MCPMCP23017_SP1.27 (GPA6); no longer MCPMCP23017_SP1.1 (GPB0)
- net ENC-SW-4: now also MCPMCP23017_SP1.28 (GPA7); no longer MCPMCP23017_SP1.4 (GPB3)
- net GND: now also C10.2, C11.2, C12.2, C14.2, C15.2, C17.2, C18.2, C20.2, C21.2, C23.2, C24.2, C25.2, C26.2, C27.2, C7.2, C8.2, C9.2, MCPMCP23017_SP2.10 (VSS), MCPMCP23017_SP2.15 (A0), MCPMCP23017_SP2.16 (A1), MCPMCP23017_SP2.17 (A2), SW10.2, SW11.2, SW12.2, SW13.2, SW14.2, SW15.2, SW16.2, SW17.2, SW18.2, SW19.2, SW20.2, SW5.2, SW6.2, SW7.2, SW8.2, SW9.2
- net SCK: now also MCPMCP23017_SP2.12 (SCK), R8.1
- net SDA: now also MCPMCP23017_SP2.13 (SDA), R7.1
- net SWITCH-1: now also MCPMCP23017_SP2.21 (GPA0); no longer MCPMCP23017_SP1.27 (GPA6)
- net SWITCH-2: now also MCPMCP23017_SP2.22 (GPA1); no longer MCPMCP23017_SP1.28 (GPA7)
- net SWITCH-3: now also MCPMCP23017_SP2.23 (GPA2); no longer MCPMCP23017_SP1.7 (GPB6)
- net SWITCH-4: now also MCPMCP23017_SP2.24 (GPA3); no longer MCPMCP23017_SP1.8 (GPB7)
- net INT3: now reaches RPi1.11 (Pin_11)
- net INT3: now also MCPMCP23017_SP1.20 (INTA)
- net INT4: now reaches RPi1.13 (Pin_13)
- net INT4: now also MCPMCP23017_SP1.19 (INTB)
- net INT1: now reaches RPi1.29 (Pin_29)
- net INT1: now also MCPMCP23017_SP2.20 (INTA)
- net INT2: now reaches RPi1.31 (Pin_31)
- net INT2: now also MCPMCP23017_SP2.19 (INTB)
- net INTA: no longer names the net of RPi1.36 (Pin_36)
- net INTA: no longer MCPMCP23017_SP1.20 (INTA)
- net INTB: no longer names the net of RPi1.37 (Pin_37)
- net INTB: no longer MCPMCP23017_SP1.19 (INTB)
- new net SWITCH-10: C14.1, MCPMCP23017_SP2.2 (GPB1), SW10.1
- new net SWITCH-11: C15.1, MCPMCP23017_SP2.3 (GPB2), SW11.1
- new net SWITCH-12: C17.1, MCPMCP23017_SP2.4 (GPB3), SW12.1
- new net SWITCH-13: C18.1, MCPMCP23017_SP2.5 (GPB4), SW13.1
- new net SWITCH-14: C20.1, MCPMCP23017_SP2.6 (GPB5), SW14.1
- new net SWITCH-15: C21.1, MCPMCP23017_SP2.7 (GPB6), SW15.1
- new net SWITCH-16: C23.1, MCPMCP23017_SP2.8 (GPB7), SW16.1
- new net SWITCH-17: C24.1, MCPMCP23017_SP1.21 (GPA0), SW17.1
- new net SWITCH-18: C25.1, MCPMCP23017_SP1.22 (GPA1), SW18.1
- new net SWITCH-19: C26.1, MCPMCP23017_SP1.23 (GPA2), SW19.1
- new net SWITCH-20: C27.1, MCPMCP23017_SP1.24 (GPA3), SW20.1
- new net SWITCH-5: C8.1, MCPMCP23017_SP2.25 (GPA4), SW5.1
- new net SWITCH-6: C9.1, MCPMCP23017_SP2.26 (GPA5), SW6.1
- new net SWITCH-7: C10.1, MCPMCP23017_SP2.27 (GPA6), SW7.1
- new net SWITCH-8: C11.1, MCPMCP23017_SP2.28 (GPA7), SW8.1
- new net SWITCH-9: C12.1, MCPMCP23017_SP2.1 (GPB0), SW9.1
- no-connect marks 37 -> 35
Other:
- note removed: "GPI02(SDA1)"
- note removed: "GPIO17(GEN0)"
- note removed: "GPIO27(GEN2)"
- note removed: "GPIO3(SCL1)"
- note removed: "GPIO5"
- note removed: "GPIO6"
- title: zynthian mini -> zynthian mini - v2 with 20 buttons
- moved on the sheet: A1, C1, C13, C16, C19, C22, C3, C31, C32, C33, C34, C4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

Commit message: first workable solution for v2 20 pins
Parts:
- RPi1: footprint Connector_PinSocket_2.54mm:PinSocket_2x20_P2.54mm_Vertical -> project-footprints:raspberry pi 4 HAT
Changed lines of the file:
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@@
 			)
 		)
-		(property "Footprint" "Connector_PinSocket_2.54mm:PinSocket_2x20_P2.54mm_Vertical"
+		(property "Footprint" "project-footprints:raspberry pi 4 HAT"
 			(at 3.81 82.55 0)
 			(effects
